Commit message: Lidar sensor fix

File: src/mobile_robot_description/urdf/lidar.xacro (robot description, xacro)
@@ -24,26 +24,35 @@
     </joint>
     <gazebo reference="lidar_link">
-        <material>Gazebo/Green</material>
-        <sensor type="ray" name="lidar_sensor">
-            <pose>0 0 0 0 0 0</pose>
-            <visualize>false</visualize>
-            <update_rate>10</update_rate>
-            <ray>
-            	<scan>
-                    <horizontal>
-                        <samples>720</samples>
-                        <resolution>1</resolution>
-                        <min_angle>-3.14</min_angle>
-                        <max_angle>3.14</max_angle>
-                    </horizontal>
-            	</scan>
-                <range>
-                    <min>0.1</min>
-                    <max>30.0</max>
-                    <resolution>0.01</resolution>
-                </range>
-            </ray>
-            <plugin name="lidar" filename="libgazebo_ros_ray_sensor.so">
-            </plugin>
+        <sensor name="lidar" type="ray">
+          <always_on>true</always_on>
+          <visualize>true</visualize>
+          <update_rate>5</update_rate>
+          <ray>
+            <scan>
+              <horizontal>
+                <samples>360</samples>
+                <resolution>1.000000</resolution>
+                <min_angle>0.000000</min_angle>
+                <max_angle>6.280000</max_angle>
+              </horizontal>
+            </scan>
+            <range>
+              <min>0.120000</min>
+              <max>3.5</max>
+              <resolution>0.015000</resolution>
+            </range>
+            <noise>
+              <type>gaussian</type>
+              <mean>0.0</mean>
+              <stddev>0.01</stddev>
+            </noise>
+          </ray>
+          <plugin name="scan" filename="libgazebo_ros_ray_sensor.so">
+            <ros>
+              <remapping>~/out:=scan</remapping>
+            </ros>
+            <output_type>sensor_msgs/LaserScan</output_type>
+            <frame_name>lidar_link</frame_name>
+          </plugin>
         </sensor>
     </gazebo>
